File: ADXRS290BCEZ_gyro/ADXRS290BCEZ_gyro.kicad_sch (KiCad schematic)
At the start: 1 part

Commit message: made some pcbs
Parts:
- added Ccp1, Cio1, Creg1, Cs1: 1u, Capacitor_SMD:C_0603_1608Metric, symbol Device:C_Small
- added U1: ~, Connector_PinHeader_2.54mm:PinHeader_1x07_P2.54mm_Vertical, symbol connectors:header
- ADXRS290BCEZ1: renamed from ADXRS290BCEZ; footprint Package_LGA:LGA-16_4x4mm_P0.65mm_LayoutBorder4x4y -> ADXRS290BCEZ:18-LFLGA
Connections:
- net at ADXRS290BCEZ1.1 (VREG): now also ADXRS290BCEZ1.17 (VREG), Creg1.1
- net at ADXRS290BCEZ1.10 (SCLK): now also U1.7 (SCLK)
- net GND: now reaches ADXRS290BCEZ1.11 (SYNC/ASEL)
- net GND: now also ADXRS290BCEZ1.13 (GND), ADXRS290BCEZ1.15 (GND), ADXRS290BCEZ1.16 (GND), Ccp1.1, Cio1.2, Creg1.2, Cs1.2, U1.1 (GND)
- net at ADXRS290BCEZ1.12 (CP): now also Ccp1.2
- net at ADXRS290BCEZ1.14 (VS): now also ADXRS290BCEZ1.18 (VS), Cs1.1, U1.3 (Vs)
- net at ADXRS290BCEZ1.2 (VDD): now also Cio1.1, U1.2 (Vdd)
- net at ADXRS290BCEZ1.7 (CS): now also U1.4 (CS)
- net at ADXRS290BCEZ1.8 (MISO): now also U1.5 (MISO)
- net at ADXRS290BCEZ1.9 (MOSI): now also U1.6 (MOSI)
- no-connect marks 0 -> 4
